Commit message: Add fake camera node

File: src/welding_robot_description/urdf/welding_robot_macro.xacro (robot description, xacro)
@@ -188,4 +188,40 @@
       <origin xyz="0.031 0.03 0.329" rpy="${radians(50)} 0 0"/>
     </joint>
+    <!-- Fixed overhead camera looking down at the workcell. -->
+    <link name="overhead_camera_link">
+      <visual>
+        <origin xyz="0 0 0" rpy="0 0 0"/>
+        <geometry>
+          <box size="0.08 0.06 0.04"/>
+        </geometry>
+        <material name="overhead_camera_green">
+          <color rgba="0.05 0.35 0.18 1.0"/>
+        </material>
+      </visual>
+      <collision>
+        <origin xyz="0 0 0" rpy="0 0 0"/>
+        <geometry>
+          <box size="0.08 0.06 0.04"/>
+        </geometry>
+      </collision>
+      <inertial>
+        <origin xyz="0 0 0" rpy="0 0 0"/>
+        <mass value="0.1"/>
+        <inertia ixx="0.00002" ixy="0.0" ixz="0.0"
+                iyy="0.00002" iyz="0.0"
+                izz="0.00002"/>
+      </inertial>
+    </link>
+    <joint name="overhead_camera_mount_joint" type="fixed">
+      <parent link="world"/>
+      <child link="overhead_camera_link"/>
+      <origin xyz="0.75 0.0 1.7" rpy="${radians(180)} 0 0"/>
+    </joint>
+    <link name="overhead_camera_optical_frame"/>
+    <joint name="overhead_camera_optical_joint" type="fixed">
+      <parent link="overhead_camera_link"/>
+      <child link="overhead_camera_optical_frame"/>
+      <origin xyz="0 0 0" rpy="0 0 0"/>
+    </joint>
     <xacro:if value="${add_ros2_control}">
       <xacro:property name="initial_positions" value="${xacro.load_yaml(initial_positions_file)['initial_positions']}"/>
