Commit message: Prepare gazebo workflow

File: src/welding_robot_bringup/urdf/welding_robot_gazebo.xacro (robot description, xacro)
@@ -13,4 +13,16 @@
     <parent link="gazebo_camera_sensor_link"/>
     <child link="gazebo_camera_optical_frame"/>
+    <origin xyz="0 0 0" rpy="${-pi/2} 0 ${-pi/2}"/>
+  </joint>
+  <link name="ee_camera_sensor_link"/>
+  <joint name="ee_camera_sensor_joint" type="fixed">
+    <parent link="welding_tcp"/>
+    <child link="ee_camera_sensor_link"/>
+    <origin xyz="0 -0.12 0" rpy="${pi} 0 ${pi/2}"/>
+  </joint>
+  <link name="ee_camera_optical_frame"/>
+  <joint name="ee_camera_optical_joint" type="fixed">
+    <parent link="ee_camera_sensor_link"/>
+    <child link="ee_camera_optical_frame"/>
     <origin xyz="0 0 0" rpy="${-pi/2} 0 ${-pi/2}"/>
   </joint>
@@ -30,4 +42,5 @@
   <gazebo reference="overhead_camera_link"><gravity>false</gravity></gazebo>
   <gazebo reference="gazebo_camera_sensor_link"><gravity>false</gravity></gazebo>
+  <gazebo reference="ee_camera_sensor_link"><gravity>false</gravity></gazebo>
   <gazebo reference="gazebo_camera_sensor_link">
     <sensor name="overhead_camera" type="camera">
@@ -55,3 +68,28 @@
     </sensor>
   </gazebo>
+  <gazebo reference="ee_camera_sensor_link">
+    <sensor name="ee_camera" type="camera">
+      <always_on>true</always_on>
+      <update_rate>30</update_rate>
+      <topic>ee_camera/image_raw</topic>
+      <visualize>false</visualize>
+      <camera>
+        <horizontal_fov>1.047</horizontal_fov>
+        <image>
+          <width>640</width>
+          <height>480</height>
+          <format>R8G8B8</format>
+        </image>
+        <clip>
+          <near>0.01</near>
+          <far>2.0</far>
+        </clip>
+        <noise>
+          <type>gaussian</type>
+          <mean>0.0</mean>
+          <stddev>0.001</stddev>
+        </noise>
+      </camera>
+    </sensor>
+  </gazebo>
 </robot>

File: src/welding_robot_bringup/urdf/welding_robot_gazebo_control.xacro (robot description, xacro)
@@ -13,4 +13,16 @@
     <parent link="gazebo_camera_sensor_link"/>
     <child link="gazebo_camera_optical_frame"/>
+    <origin xyz="0 0 0" rpy="${-pi/2} 0 ${-pi/2}"/>
+  </joint>
+  <link name="ee_camera_sensor_link"/>
+  <joint name="ee_camera_sensor_joint" type="fixed">
+    <parent link="welding_tcp"/>
+    <child link="ee_camera_sensor_link"/>
+    <origin xyz="0 -0.12 0" rpy="${pi} 0 ${pi/2}"/>
+  </joint>
+  <link name="ee_camera_optical_frame"/>
+  <joint name="ee_camera_optical_joint" type="fixed">
+    <parent link="ee_camera_sensor_link"/>
+    <child link="ee_camera_optical_frame"/>
     <origin xyz="0 0 0" rpy="${-pi/2} 0 ${-pi/2}"/>
   </joint>
@@ -113,3 +125,28 @@
     </sensor>
   </gazebo>
+  <gazebo reference="ee_camera_sensor_link">
+    <sensor name="ee_camera" type="camera">
+      <always_on>true</always_on>
+      <update_rate>30</update_rate>
+      <topic>ee_camera/image_raw</topic>
+      <visualize>false</visualize>
+      <camera>
+        <horizontal_fov>1.047</horizontal_fov>
+        <image>
+          <width>640</width>
+          <height>480</height>
+          <format>R8G8B8</format>
+        </image>
+        <clip>
+          <near>0.01</near>
+          <far>2.0</far>
+        </clip>
+        <noise>
+          <type>gaussian</type>
+          <mean>0.0</mean>
+          <stddev>0.001</stddev>
+        </noise>
+      </camera>
+    </sensor>
+  </gazebo>
 </robot>

File: src/welding_robot_description/urdf/welding_robot_macro.xacro (robot description, xacro)
@@ -216,5 +216,5 @@
       <parent link="world"/>
       <child link="overhead_camera_link"/>
-      <origin xyz="0.75 0.0 1.7" rpy="${radians(180)} 0 0"/>
+      <origin xyz="0.6 0.0 2.2" rpy="${radians(180)} 0 0"/>
     </joint>
     <link name="overhead_camera_optical_frame"/>
